File: hardware/cg2111a_robot_kicad/cg2111a_robot.kicad_sch (KiCad schematic)
At the start: 11 parts, among them J1 Conn_01x04_Pin, J2 Conn_01x04_Pin, J3 Conn_01x05, J4 Conn_01x05, J5 Conn_01x03, J6 Conn_01x03, Q1 2N3904, U3 RASPBERRY_PI_4B_4GB

Commit message: final edits for final run
Other:
- note added: "Extra Ultrasonic Port that was not used"
Changed lines of the file:
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@@
     (effects (font (face "Consolas") (size 5 5) bold) (justify left bottom))
+  )
+  (text "Extra Ultrasonic Port \nthat was not used\n" (at 223.52 67.31 0)
+    (effects (font (size 1.27 1.27)) (justify left bottom))
   )
   (text "Motor Shield connected to the Arduino\nMotors are connected to the Shield"

Commit message: updates and stuff
Parts:
- removed J2: Conn_01x04_Pin, symbol Connector_Generic:Conn_01x04
Other:
- note removed: "Extra Ultrasonic Port that was not used"
- moved on the sheet: J3, J4, J5, J6
